File: RS485-CH340E.kicad_sch (KiCad schematic)
At the start: 13 parts, among them J1 USB_A, J2 Conn_01x04_Pin, J3 Conn_02x04_Odd_Even, U1 NCP1117-3.3_SOT223, U2 SP3485CN, U3 CH340E

Commit message: Update to CH340X chip (more modern) Regenerate front/back/pcb.png files
Parts:
- removed U3: CH340E, Package_SO:MSOP-10_3x3mm_P0.5mm, symbol Interface_USB:CH340E
- added C5: 100nF, Capacitor_SMD:C_0603_1608Metric, symbol Device:C
- added U3: CH340X, Package_SO:MSOP-10_3x3mm_P0.5mm, symbol Interface_USB:CH340X
Connections:
- net GND1 is gone; now on net GND: C4.2
- net GND: now also C5.2, U3.3 (GND)
- net RxD: now also U3.9 (RXD)
- net TXE: now also U3.6 (TNOW/~{DTR})
- net TxD: now also U3.8 (TXD)
- net VCC: now also U3.7 (VCC)
- net at J1.2 (D-): now also U3.2 (UD-)
- net at J1.3 (D+): now also U3.1 (UD+)
- new net: C5.1, U3.10 (V3)
